File: PCB/rgbleds.sch (KiCad schematic (older format))
At the start: 62 parts

Commit message: Updates to the PCB
Parts:
- D100, D101, D102, D103, D104, D105, D106, D107, D108, D109, D110, D111, D112, D113, D114, D115, D116, D117, D118, D119, D120, D121, D122, D123, D124, D125, D64, D65, D66, D67, D68, D69, D70, D71, D72, D73, D74, D75, D76, D77, D78, D79, D80, D81, D82, D83, D84, D85, D86, D87, D88, D89, D90, D91, D92, D93, D94, D95, D96, D97, D98, D99: renamed from D?; value LED_RGBA -> LED_RAGB; footprint (none) -> LED_THT:LED_D5.0mm-4_RGB_Wide_Pins; symbol Device:LED_RGBA -> Device:LED_RAGB
Connections:
- net CS1: now also D102.2 (A), D64.2 (A), D76.2 (A), D89.2 (A); no longer D102.4 (A), D64.4 (A), D76.4 (A), D89.4 (A)
- net CS10: now also D111.2 (A), D73.2 (A), D85.2 (A), D98.2 (A); no longer D111.4 (A), D73.4 (A), D85.4 (A), D98.4 (A)
- net CS11: now also D112.2 (A), D74.2 (A), D86.2 (A), D99.2 (A); no longer D112.4 (A), D74.4 (A), D86.4 (A), D99.4 (A)
- net CS12: now also D100.2 (A), D113.2 (A), D75.2 (A), D87.2 (A); no longer D100.4 (A), D113.4 (A), D119.4 (A), D122.4 (A), D125.4 (A), D75.4 (A), D87.4 (A)
- net CS13: now also D101.2 (A), D88.2 (A); no longer D101.4 (A), D102.1 (RK), D102.2 (GK), D102.3 (BK), D103.1 (RK), D103.2 (GK), D103.3 (BK), D104.1 (RK), D104.2 (GK), D104.3 (BK), D105.1 (RK), D105.2 (GK), D105.3 (BK), D106.1 (RK), D106.2 (GK), D106.3 (BK), D107.1 (RK), D107.2 (GK), D107.3 (BK), D108.1 (RK), D108.2 (GK), D108.3 (BK), D109.1 (RK), D109.2 (GK), D109.3 (BK), D110.1 (RK), D110.2 (GK), D110.3 (BK), D111.1 (RK), D111.2 (GK), D111.3 (BK), D112.1 (RK), D112.2 (GK), D112.3 (BK), D113.1 (RK), D113.2 (GK), D113.3 (BK), D114.1 (RK), D114.3 (BK), D114.4 (A), D115.1 (RK), D115.2 (GK), D115.3 (BK), D116.1 (RK), D116.2 (GK), D116.3 (BK), D116.4 (A), D118.4 (A), D121.4 (A), D124.4 (A), D88.4 (A)
- net CS14: now also D115.2 (A), D118.2 (A), D121.2 (A), D124.2 (A); no longer D115.4 (A), D117.4 (A), D120.4 (A), D123.4 (A)
- net CS2: now also D103.2 (A), D65.2 (A), D77.2 (A), D90.2 (A); no longer D103.4 (A), D65.4 (A), D77.4 (A), D90.4 (A)
- net CS3: now also D104.2 (A), D66.2 (A), D78.2 (A), D91.2 (A); no longer D104.4 (A), D66.4 (A), D78.4 (A), D91.4 (A)
- net CS4: now also D105.2 (A), D67.2 (A), D79.2 (A), D92.2 (A); no longer D105.4 (A), D67.4 (A), D79.4 (A), D92.4 (A)
- net CS5: now also D106.2 (A), D68.2 (A), D80.2 (A), D93.2 (A); no longer D106.4 (A), D68.4 (A), D80.4 (A), D93.4 (A)
- net CS6: now also D107.2 (A), D69.2 (A), D81.2 (A), D94.2 (A); no longer D107.4 (A), D69.4 (A), D81.4 (A), D94.4 (A)
- net CS7: now also D108.2 (A), D70.2 (A), D82.2 (A), D95.2 (A); no longer D108.4 (A), D70.4 (A), D82.4 (A), D95.4 (A)
- net CS8: now also D109.2 (A), D71.2 (A), D83.2 (A), D96.2 (A); no longer D109.4 (A), D71.4 (A), D83.4 (A), D96.4 (A)
- net CS9: now also D110.2 (A), D72.2 (A), D84.2 (A), D97.2 (A); no longer D110.4 (A), D72.4 (A), D84.4 (A), D97.4 (A)
- net SW10: now also D124.4 (BK), D125.4 (BK), D64.4 (BK), D65.4 (BK), D66.4 (BK), D67.4 (BK), D68.4 (BK), D69.4 (BK), D70.4 (BK), D71.4 (BK), D72.4 (BK), D73.4 (BK), D74.4 (BK), D75.4 (BK); no longer D123.3 (BK), D124.3 (BK), D125.3 (BK), D64.3 (BK), D65.3 (BK), D66.3 (BK), D67.3 (BK), D68.3 (BK), D69.3 (BK), D70.3 (BK), D71.3 (BK), D72.3 (BK), D73.3 (BK), D74.3 (BK), D75.3 (BK)
- net SW11: now also D124.3 (GK), D125.3 (GK), D64.3 (GK), D65.3 (GK), D66.3 (GK), D67.3 (GK), D68.3 (GK), D69.3 (GK), D70.3 (GK), D71.3 (GK), D72.3 (GK), D73.3 (GK), D74.3 (GK), D75.3 (GK); no longer D123.2 (GK), D124.2 (GK), D125.2 (GK), D64.2 (GK), D65.2 (GK), D66.2 (GK), D67.2 (GK), D68.2 (GK), D69.2 (GK), D70.2 (GK), D71.2 (GK), D72.2 (GK), D73.2 (GK), D74.2 (GK), D75.2 (GK)
- net SW12: no longer D123.1 (RK)
- net SW4: now also D100.4 (BK), D101.4 (BK), D118.4 (BK), D119.4 (BK), D120.4 (BK), D89.4 (BK), D90.4 (BK), D91.4 (BK), D92.4 (BK), D93.4 (BK), D94.4 (BK), D95.4 (BK), D96.4 (BK), D97.4 (BK), D98.4 (BK), D99.4 (BK); no longer D100.3 (BK), D101.3 (BK), D117.3 (BK), D118.3 (BK), D119.3 (BK), D89.3 (BK), D90.3 (BK), D91.3 (BK), D92.3 (BK), D93.3 (BK), D94.3 (BK), D95.3 (BK), D96.3 (BK), D97.3 (BK), D98.3 (BK), D99.3 (BK)
- net SW5: now also D100.3 (GK), D101.3 (GK), D118.3 (GK), D119.3 (GK), D120.3 (GK), D89.3 (GK), D90.3 (GK), D91.3 (GK), D92.3 (GK), D93.3 (GK), D94.3 (GK), D95.3 (GK), D96.3 (GK), D97.3 (GK), D98.3 (GK), D99.3 (GK); no longer D100.2 (GK), D101.2 (GK), D117.2 (GK), D118.2 (GK), D119.2 (GK), D89.2 (GK), D90.2 (GK), D91.2 (GK), D92.2 (GK), D93.2 (GK), D94.2 (GK), D95.2 (GK), D96.2 (GK), D97.2 (GK), D98.2 (GK), D99.2 (GK)
- net SW6: now also D120.1 (RK); no longer D117.1 (RK)
- net SW7: now also D121.4 (BK), D122.4 (BK), D123.4 (BK), D76.4 (BK), D77.4 (BK), D78.4 (BK), D79.4 (BK), D80.4 (BK), D81.4 (BK), D82.4 (BK), D83.4 (BK), D84.4 (BK), D85.4 (BK), D86.4 (BK), D87.4 (BK), D88.4 (BK); no longer D120.3 (BK), D121.3 (BK), D122.3 (BK), D76.3 (BK), D77.3 (BK), D78.3 (BK), D79.3 (BK), D80.3 (BK), D81.3 (BK), D82.3 (BK), D83.3 (BK), D84.3 (BK), D85.3 (BK), D86.3 (BK), D87.3 (BK), D88.3 (BK)
- net SW8: now also D121.3 (GK), D122.3 (GK), D123.3 (GK), D76.3 (GK), D77.3 (GK), D78.3 (GK), D79.3 (GK), D80.3 (GK), D81.3 (GK), D82.3 (GK), D83.3 (GK), D84.3 (GK), D85.3 (GK), D86.3 (GK), D87.3 (GK), D88.3 (GK); no longer D120.2 (GK), D121.2 (GK), D122.2 (GK), D76.2 (GK), D77.2 (GK), D78.2 (GK), D79.2 (GK), D80.2 (GK), D81.2 (GK), D82.2 (GK), D83.2 (GK), D84.2 (GK), D85.2 (GK), D86.2 (GK), D87.2 (GK), D88.2 (GK)
- net SW9: now also D123.1 (RK); no longer D120.1 (RK)
- new net CS15: D116.2 (A), D119.2 (A), D122.2 (A), D125.2 (A)
- new net CS16: D117.2 (A), D120.2 (A), D123.2 (A)
- new net SW1: D102.4 (BK), D103.4 (BK), D104.4 (BK), D105.4 (BK), D106.4 (BK), D107.4 (BK), D108.4 (BK), D109.4 (BK), D110.4 (BK), D111.4 (BK), D112.4 (BK), D113.4 (BK), D114.4 (BK), D115.4 (BK), D116.4 (BK), D117.4 (BK)
- new net SW2: D102.3 (GK), D103.3 (GK), D104.3 (GK), D105.3 (GK), D106.3 (GK), D107.3 (GK), D108.3 (GK), D109.3 (GK), D110.3 (GK), D111.3 (GK), D112.3 (GK), D113.3 (GK), D114.3 (GK), D115.3 (GK), D116.3 (GK), D117.3 (GK)
- new net SW3: D102.1 (RK), D103.1 (RK), D104.1 (RK), D105.1 (RK), D106.1 (RK), D107.1 (RK), D108.1 (RK), D109.1 (RK), D110.1 (RK), D111.1 (RK), D112.1 (RK), D113.1 (RK), D114.1 (RK), D115.1 (RK), D117.1 (RK)
