File: PCB/ULK.kicad_pcb (KiCad board)
At the start: 2 copper layers, 226 parts, among them J1 AVR-ISP-6, K1 SW_Push, K10 SW_Push, K11 SW_Push, K12 SW_Push, K13 SW_Push, K14 SW_Push, K15 SW_Push, K16 SW_Push, K17 SW_Push, K18 SW_Push, K19 SW_Push, K2 SW_Push, K20 SW_Push, K21 SW_Push, K22 SW_Push, K23 SW_Push, K24 SW_Push, K25 SW_Push, K26 SW_Push, K27 SW_Push, K28 SW_Push, K29 SW_Push, K3 SW_Push, K30 SW_Push, K31 SW_Push, K32 SW_Push, K33 SW_Push, K34 SW_Push, K35 SW_Push, K36 SW_Push, K37 SW_Push, K38 SW_Push, K39 SW_Push, K4 SW_Push, K40 SW_Push, K41 SW_Push, K42 SW_Push, K43 SW_Push, K44 SW_Push, K45 SW_Push, K46 SW_Push, K47 SW_Push, K48 SW_Push, K49 SW_Push, K5 SW_Push, K50 SW_Push, K51 SW_Push, K52 SW_Push, K53 SW_Push, K54 SW_Push, K55 SW_Push, K56 SW_Push, K57 SW_Push, K58 SW_Push, K59 SW_Push, K6 SW_Push, K60 SW_Push, K61 SW_Push, K62 SW_Push, K7 SW_Push, K8 SW_Push, K9 SW_Push, SW1 SW_Push, SW2 Rotary_Encoder_Switch, U1 PRTR5V0U2X, U2 ATmega32U4-MU, U3 IS31FL3733-QF, Y1 XTAL

Commit message: PCB to the tracing stage
Parts:
- C1, C10, C11, C12, C13, C14, C15, C16, C2, C3, C4, C5, C6, C7, C8, C9, F1, J1, R1, R10, R11, R12, R2, R3, R4, R5, R6, R7, R8, R9, SW1, U1, USB1, Y1: moved to B.Cu
- K58: footprint MX_Only:MXOnly-2U-NoLED -> MX_Only:MXOnly-1U-NoLED
- moved R3 222.1 mm to (81.6, 31.8), turned to 180 degrees
- moved U1 218.9 mm to (84.9, 34.9), turned to 180 degrees
- moved R4 205.6 mm to (87.3, 31.8)
- moved F1 189.2 mm to (92.1, 32.4), turned to 90 degrees
- moved C2 189.0 mm to (110.3, 30.2), turned to 90 degrees
- moved C1 178.9 mm to (100.8, 30.3), turned to 270 degrees
- moved Y1 174.0 mm to (105.6, 30.2)
- moved J1 159.1 mm to (130.2, 17.5)
- moved SW1 152.4 mm to (130.2, 7.94), turned to 90 degrees
- moved R1 127.8 mm to (170.5, 36.5), turned to 180 degrees
- moved R2 124.6 mm to (170.5, 34.1), turned to 180 degrees
- moved C4 123.9 mm to (175.4, 26.8), turned to 90 degrees
- moved R5 122.0 mm to (181.8, 25.3), turned to 270 degrees
- moved R6 119.8 mm to (187.3, 34.8), turned to 90 degrees
- moved C14 118.0 mm to (183.2, 40.5), turned to 180 degrees
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Connections:
- net Net-(R1-Pad2) renamed DN
- net Net-(R2-Pad2) renamed DP
Routing:
- net SW8: track 0.00 -> 261.7 mm, vias 0 -> 11
- net SW9: track 0.00 -> 244.8 mm
- net Row2: track 0.00 -> 244.2 mm
- net Row3: track 0.00 -> 244.2 mm
- net Row1: track 0.00 -> 244.2 mm
- net Row0: track 0.00 -> 243.2 mm
- net Row4: track 0.00 -> 241.5 mm
- net SW11: track 0.00 -> 241.1 mm, vias 0 -> 10
- net SW7: track 0.00 -> 240.8 mm
- net SW12: track 0.00 -> 224.4 mm
- net SW10: track 0.00 -> 220.8 mm
- net DP: track 0.00 -> 101.2 mm
- net DN: track 0.00 -> 100.9 mm
- net Col5: track 0.00 -> 86.1 mm
- net Col4: track 0.00 -> 84.1 mm
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Other:
- board outline added: 247.6 x 117.5 mm
- net class Power added: clearance 0.2, trace_width 0.381, via_dia 0.8, via_drill 0.4
