File: PCB/ULK.sch (KiCad schematic (older format))
At the start: 36 parts

Commit message: Updates to the PCB
Parts:
- removed U?: ATmega32U4-AU, Package_QFP:TQFP-44_10x10mm_P0.8mm, symbol MCU_Microchip_ATmega:ATmega32U4-AU
- added U2: ATmega32U4-MU, Package_DFN_QFN:QFN-44-1EP_7x7mm_P0.5mm_EP5.2x5.2mm, symbol MCU_Microchip_ATmega:ATmega32U4-MU
- C1, C10, C11, C12, C13, C14, C15, C16, C2, C5, C6, C7, C8, C9: renamed from C?; footprint (none) -> Capacitor_SMD:C_0805_2012Metric
- C3: renamed from C?; footprint (none) -> Capacitor_Tantalum_SMD:CP_EIA-3216-18_Kemet-A
- C4: renamed from C7; footprint (none) -> Capacitor_SMD:C_0805_2012Metric
- F1: renamed from F?; footprint (none) -> Fuse:Fuse_1206_3216Metric
- J1: renamed from J?; footprint (none) -> random-keyboard-parts:Reset_Pretty-Mask
- R1, R10, R11, R12, R2, R3, R4, R5, R6, R7, R8, R9: renamed from R?; footprint (none) -> Resistor_SMD:R_0805_2012Metric
- SW1: renamed from SW?; footprint (none) -> Button_Switch_SMD:SW_SPST_SKQG_WithStem
- U1: renamed from U?; footprint (none) -> random-keyboard-parts:SOT143B
- U3: renamed from U?; value IS31FL3733-TQ -> IS31FL3733-QF; footprint Package_QFP:TQFP-48-1EP_7x7mm_P0.5mm_EP5x5mm -> Package_DFN_QFN:QFN-48-1EP_6x6mm_P0.4mm_EP4.2x4.2mm; symbol Driver_LED:IS31FL3733-TQ -> Driver_LED:IS31FL3733-QF
- USB1: renamed from USB?; footprint (none) -> Type-C:HRO-TYPE-C-31-M-12-HandSoldering
- Y1: renamed from Y?; footprint (none) -> Crystal:Crystal_SMD_3225-4Pin_3.2x2.5mm
Connections:
- net +5V: now also U2.14 (VCC), U2.2 (UVCC), U2.24 (AVCC), U2.34 (VCC), U2.44 (AVCC), U2.7 (VBUS)
- net Col0: now also U2.20 (PD2)
- net Col1: now also U2.21 (PD3)
- net Col10: now also U2.40 (PF1)
- net Col11: now also U2.41 (PF0)
- net Col12: now also U2.1 (PE6)
- net Col2: now also U2.25 (PD4)
- net Col3: now also U2.22 (PD5)
- net Col4: now also U2.26 (PD6)
- net Col5: now also U2.27 (PD7)
- net Col6: now also U2.36 (PF7)
- net Col7: now also U2.37 (PF6)
- net Col8: now also U2.38 (PF5)
- net Col9: now also U2.39 (PF4)
- net D+: now also U2.4 (D+)
- net D-: now also U2.3 (D-)
- net GND: now also U2.15 (GND), U2.23 (GND), U2.35 (GND), U2.43 (GND), U2.45 (GND), U2.5 (UGND)
- net MISO: now also U2.11 (PB3)
- net MOSI: now also U2.10 (PB2)
- net RESET: now also U2.13 (~RESET)
- net Rot0: now also U2.12 (PB7)
- net Rot1: now also U2.8 (PB0)
- net Row0: now also U2.28 (PB4)
- net Row1: now also U2.29 (PB5)
- net Row2: now also U2.30 (PB6)
- net Row3: now also U2.31 (PC6)
- net Row4: now also U2.32 (PC7)
- net SCK: now also U2.9 (PB1)
- net SCL: now also U2.18 (PD0)
- net SDA: now also U2.19 (PD1)
- net VCC: now also C11.2, R7.1, R8.1, R9.1, U3.39 (VIO)
- net XTAL1: now also U2.17 (XTAL1)
- net XTAL2: now also U2.16 (XTAL2)
- net at R6.2: now also U2.33 (~HWB~/PE2)
- net at C4.1: now also U2.6 (UCAP)
- no-connect marks 3 -> 4

Commit message: PCB to the tracing stage
Connections:
- net DN: now reaches R1.2, U1.3 (IO2), USB1.5 (DN2), USB1.7 (DN1)
- net DP: now reaches R2.2, U1.2 (IO1), USB1.6 (DP1), USB1.8 (DP2)
Changed lines of the file:
@@
 	9500 1500 9400 1500
 Connection ~ 9400 1500
+Text GLabel 5100 2300 3    50   Input ~ 0
+DP
+Text GLabel 5100 2200 1    50   Input ~ 0
+DN
 $EndSCHEMATC
