File: PCB/matrix.sch (KiCad schematic (older format))
At the start: 128 parts

Commit message: Updates to the PCB
Parts:
- C17, C18: renamed from C?; footprint (none) -> Capacitor_SMD:C_0805_2012Metric
- D1, D10, D11, D12, D13, D14, D15, D16, D17, D18, D19, D2, D20, D21, D22, D23, D24, D25, D26, D27, D28, D29, D3, D30, D31, D32, D33, D34, D35, D36, D37, D38, D39, D4, D40, D41, D42, D43, D44, D45, D46, D47, D48, D49, D5, D50, D51, D52, D53, D54, D55, D56, D57, D58, D59, D6, D60, D61, D62, D63, D7, D8, D9: renamed from D?; footprint (none) -> Diode_SMD:D_SOD-123
- K1, K10, K11, K12, K13, K14, K15, K16, K17, K18, K19, K2, K20, K21, K22, K23, K24, K25, K26, K27, K28, K29, K3, K30, K31, K32, K33, K34, K35, K36, K37, K38, K39, K4, K40, K41, K42, K43, K44, K45, K46, K47, K48, K49, K5, K50, K51, K52, K53, K54, K6, K60, K61, K62, K7, K8, K9: renamed from K?; footprint (none) -> MX_Only:MXOnly-1U-NoLED
- K55, K56, K57, K59: renamed from K?; footprint (none) -> MX_Only:MXOnly-1.25U-NoLED
- K58: renamed from K?; footprint (none) -> MX_Only:MXOnly-2U-NoLED
- SW2: renamed from SW?; footprint (none) -> Rotary_Encoder:RotaryEncoder_Alps_EC11E-Switch_Vertical_H20mm

Commit message: PCB to the tracing stage
Parts:
- K58: footprint MX_Only:MXOnly-2U-NoLED -> MX_Only:MXOnly-1U-NoLED
Changed lines of the file:
@@
 F 0 "K58" H 6350 5243 50  0000 C CNN
 F 1 "SW_Push" H 6350 5244 50  0001 C CNN
-F 2 "MX_Only:MXOnly-2U-NoLED" H 6350 5250 50  0001 C CNN
+F 2 "MX_Only:MXOnly-1U-NoLED" H 6350 5250 50  0001 C CNN
 F 3 "~" H 6350 5250 50  0001 C CNN
 	1    6350 5050
